File: Hardware/SparkFun_Motor_Driver-TB6612FNG_v11.brd (EAGLE design)
At the start: 20.3 x 20.3 mm, 14 parts, among them U1 TB6612FNG

Commit message: changed header
Parts:
- JP1, JP2: device Testing:1X08_OFFSET_SMALL -> Testing:1X01_OFFSET_SMALL
Connections:
- net A01: now also JP1.P$5; no longer JP1.5
- net A02: now also JP1.P$4; no longer JP1.4
- net AIN1: now also JP2.P$3; no longer JP2.3
- net AIN2: now also JP2.P$2; no longer JP2.2
- net B01: now also JP1.P$2; no longer JP1.2
- net B02: now also JP1.P$3; no longer JP1.3
- net BIN1: now also JP2.P$5; no longer JP2.5
- net BIN2: now also JP2.P$6; no longer JP2.6
- net GND: now also JP1.P$1, JP1.P$6, JP2.P$8; no longer JP1.1, JP1.6, JP2.8
- net PWMA: now also JP2.P$1; no longer JP2.1
- net PWMB: now also JP2.P$7; no longer JP2.7
- net STBY: now also JP2.P$4; no longer JP2.4
- net VCC: now also JP1.P$7; no longer JP1.7
- net VM: now also JP1.P$8; no longer JP1.8
Changed lines of the file:
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@@
 <layer number="27" name="tValues" color="7" fill="1" visible="no" active="yes"/>
 <layer number="28" name="bValues" color="7" fill="1" visible="no" active="yes"/>
-<layer number="29" name="tStop" color="7" fill="3" visible="no" active="yes"/>
-<layer number="30" name="bStop" color="7" fill="6" visible="no" active="yes"/>
+<layer number="29" name="tStop" color="7" fill="3" visible="yes" active="yes"/>
+<layer number="30" name="bStop" color="7" fill="6" visible="yes" active="yes"/>
 <layer number="31" name="tCream" color="7" fill="4" visible="no" active="yes"/>
 <layer number="32" name="bCream" color="7" fill="5" visible="no" active="yes"/>
@@
 <attribute name="VALUE" x="14.704" y="24.2" size="1.016" layer="27" rot="R180"/>
 </element>
-<element name="JP1" library="Testing" package="1X08_OFFSET_SMALL" value="" x="2.54" y="1.27" smashed="yes" rot="R90">
+<element name="JP1" library="Testing" package="1X01_OFFSET_SMALL" value="" x="2.54" y="1.27" smashed="yes" rot="R90">
 <attribute name="VALUE" x="6.35" y="0" size="1.27" layer="27" rot="R90"/>
 </element>
-<element name="JP2" library="Testing" package="1X08_OFFSET_SMALL" value="" x="17.78" y="19.05" smashed="yes" rot="R270">
+<element name="JP2" library="Testing" package="1X01_OFFSET_SMALL" value="" x="17.78" y="19.05" smashed="yes" rot="R270">
 <attribute name="VALUE" x="13.97" y="20.32" size="1.27" layer="27" rot="R270"/>
 </element>
@@
 <contactref element="C3" pad="C"/>
 <contactref element="C2" pad="2"/>
-<contactref element="JP1" pad="1"/>
-<contactref element="JP2" pad="8"/>
-<contactref element="JP1" pad="6"/>
+<contactref element="JP1" pad="P$1"/>
+<contactref element="JP2" pad="P$8"/>
+<contactref element="JP1" pad="P$6"/>
 <wire x1="6.504" y1="6.615" x2="6.504" y2="7.265" width="0.254" layer="1"/>
 <wire x1="6.504" y1="10.515" x2="6.504" y2="11.165" width="0.254" layer="1"/>
@@
 <contactref element="U1" pad="2"/>
 <contactref element="U1" pad="1"/>
-<contactref element="JP1" pad="5"/>
+<contactref element="JP1" pad="P$5"/>
 <wire x1="6.35" y1="12.1412" x2="6.7564" y2="12.1412" width="0.9144" layer="1"/>
 <wire x1="6.7564" y1="12.1412" x2="6.7818" y2="12.1158" width="0.9144" layer="1"/>
@@
 <contactref element="U1" pad="6"/>
 <contactref element="U1" pad="5"/>
-<contactref element="JP1" pad="4"/>
+<contactref element="JP1" pad="P$4"/>
 <wire x1="6.35" y1="9.5504" x2="6.7564" y2="9.5504" width="0.9144" layer="1"/>
 <wire x1="6.7564" y1="9.5504" x2="6.7818" y2="9.525" width="0.9144" layer="1"/>
@@
 <contactref element="U1" pad="8"/>
 <contactref element="U1" pad="7"/>
-<contactref element="JP1" pad="3"/>
+<contactref element="JP1" pad="P$3"/>
 <wire x1="6.35" y1="8.2296" x2="6.7818" y2="8.2296" width="0.9144" layer="1"/>
 <wire x1="6.504" y1="8.0756" x2="6.504" y2="7.915" width="0.254" layer="1"/>
@@
 <contactref element="U1" pad="12"/>
 <contactref element="U1" pad="11"/>
-<contactref element="JP1" pad="2"/>
+<contactref element="JP1" pad="P$2"/>
 <wire x1="6.35" y1="5.6388" x2="6.7818" y2="5.6388" width="0.9144" layer="1"/>
 <wire x1="6.504" y1="5.4848" x2="6.504" y2="5.315" width="0.254" layer="1"/>
@@
 <contactref element="C1" pad="1"/>
 <contactref element="C3" pad="A"/>
-<contactref element="JP1" pad="8"/>
+<contactref element="JP1" pad="P$8"/>
 <wire x1="8.89" y1="16.51" x2="8.51" y2="16.51" width="0.9144" layer="1"/>
 <wire x1="10.668" y1="14.732" x2="8.89" y2="16.51" width="0.9144" layer="1"/>
@@
 <signal name="VCC">
 <contactref element="U1" pad="20"/>
-<contactref element="JP1" pad="7"/>
+<contactref element="JP1" pad="P$7"/>
 <contactref element="C2" pad="1"/>
 <wire x1="9.54" y1="13.97" x2="9.54" y2="14.59" width="0.254" layer="1"/>
@@
 <signal name="PWMA">
 <contactref element="U1" pad="23"/>
-<contactref element="JP2" pad="1"/>
+<contactref element="JP2" pad="P$1"/>
 <wire x1="13.816" y1="11.815" x2="14.609" y2="11.815" width="0.254" layer="1"/>
 <wire x1="14.609" y1="11.815" x2="14.9606" y2="12.1666" width="0.254" layer="1"/>
@@
 <signal name="AIN2">
 <contactref element="U1" pad="22"/>
-<contactref element="JP2" pad="2"/>
+<contactref element="JP2" pad="P$2"/>
 <wire x1="13.816" y1="11.165" x2="14.848" y2="11.165" width="0.254" layer="1"/>
 <wire x1="14.848" y1="11.165" x2="15.494" y2="11.811" width="0.254" layer="1"/>
@@
 <signal name="AIN1">
 <contactref element="U1" pad="21"/>
-<contactref element="JP2" pad="3"/>
+<contactref element="JP2" pad="P$3"/>
 <wire x1="13.97" y1="13.97" x2="17.78" y2="13.97" width="0.254" layer="16"/>
 <wire x1="12.2682" y1="12.2682" x2="13.97" y2="13.97" width="0.254" layer="16"/>
@@
 <signal name="STBY">
 <contactref element="U1" pad="19"/>
-<contactref element="JP2" pad="4"/>
+<contactref element="JP2" pad="P$4"/>
 <wire x1="13.816" y1="9.215" x2="14.676" y2="9.215" width="0.254" layer="1"/>
 <wire x1="14.676" y1="9.215" x2="15.24" y2="9.779" width="0.254" layer="1"/>
@@
 <signal name="BIN1">
 <contactref element="U1" pad="17"/>
-<contactref element="JP2" pad="5"/>
+<contactref element="JP2" pad="P$5"/>
 <wire x1="13.816" y1="7.915" x2="14.9" y2="7.915" width="0.254" layer="1"/>
 <wire x1="14.9" y1="7.915" x2="15.875" y2="8.89" width="0.254" layer="1"/>
@@
 <signal name="BIN2">
 <contactref element="U1" pad="16"/>
-<contactref element="JP2" pad="6"/>
+<contactref element="JP2" pad="P$6"/>
 <wire x1="13.816" y1="7.265" x2="15.595" y2="7.265" width="0.254" layer="1"/>
 <wire x1="15.595" y1="7.265" x2="16.51" y2="6.35" width="0.254" layer="1"/>
@@
 <signal name="PWMB">
 <contactref element="U1" pad="15"/>
-<contactref element="JP2" pad="7"/>
+<contactref element="JP2" pad="P$7"/>
 <wire x1="13.816" y1="6.615" x2="14.975" y2="6.615" width="0.254" layer="1"/>
 <wire x1="14.975" y1="6.615" x2="15.24" y2="6.35" width="0.254" layer="1"/>

Commit message: updated part lbr
Parts:
- JP1, JP2: device Testing:1X01_OFFSET_SMALL -> Testing:1X08_OFFSET_REDUCED
Connections:
- net A01: now also JP1.5; no longer JP1.P$5
- net A02: now also JP1.4; no longer JP1.P$4
- net AIN1: now also JP2.3; no longer JP2.P$3
- net AIN2: now also JP2.2; no longer JP2.P$2
- net B01: now also JP1.2; no longer JP1.P$2
- net B02: now also JP1.3; no longer JP1.P$3
- net BIN1: now also JP2.5; no longer JP2.P$5
- net BIN2: now also JP2.6; no longer JP2.P$6
- net GND: now also JP1.1, JP1.6, JP2.8; no longer JP1.P$1, JP1.P$6, JP2.P$8
- net PWMA: now also JP2.1; no longer JP2.P$1
- net PWMB: now also JP2.7; no longer JP2.P$7
- net STBY: now also JP2.4; no longer JP2.P$4
- net VCC: now also JP1.7; no longer JP1.P$7
- net VM: now also JP1.8; no longer JP1.P$8
Changed lines of the file:
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@@
 <layer number="20" name="Dimension" color="15" fill="1" visible="yes" active="yes"/>
 <layer number="21" name="tPlace" color="16" fill="1" visible="yes" active="yes"/>
-<layer number="22" name="bPlace" color="14" fill="1" visible="yes" active="yes"/>
+<layer number="22" name="bPlace" color="14" fill="1" visible="no" active="yes"/>
 <layer number="23" name="tOrigins" color="15" fill="1" visible="yes" active="yes"/>
-<layer number="24" name="bOrigins" color="15" fill="1" visible="yes" active="yes"/>
-<layer number="25" name="tNames" color="7" fill="1" visible="no" active="yes"/>
+<layer number="24" name="bOrigins" color="15" fill="1" visible="no" active="yes"/>
+<layer number="25" name="tNames" color="7" fill="1" visible="yes" active="yes"/>
 <layer number="26" name="bNames" color="7" fill="1" visible="no" active="yes"/>
 <layer number="27" name="tValues" color="7" fill="1" visible="no" active="yes"/>
 <layer number="28" name="bValues" color="7" fill="1" visible="no" active="yes"/>
-<layer number="29" name="tStop" color="7" fill="3" visible="yes" active="yes"/>
-<layer number="30" name="bStop" color="7" fill="6" visible="yes" active="yes"/>
+<layer number="29" name="tStop" color="7" fill="3" visible="no" active="yes"/>
+<layer number="30" name="bStop" color="7" fill="6" visible="no" active="yes"/>
 <layer number="31" name="tCream" color="7" fill="4" visible="no" active="yes"/>
 <layer number="32" name="bCream" color="7" fill="5" visible="no" active="yes"/>
@@
 <layer number="42" name="bRestrict" color="1" fill="10" visible="no" active="yes"/>
 <layer number="43" name="vRestrict" color="2" fill="10" visible="no" active="yes"/>
-<layer number="44" name="Drills" color="7" fill="1" visible="no" active="yes"/>
+<layer number="44" name="Drills" color="7" fill="1" visible="yes" active="yes"/>
 <layer number="45" name="Holes" color="7" fill="1" visible="yes" active="yes"/>
 <layer number="46" name="Milling" color="3" fill="1" visible="no" active="yes"/>
@@
 <layer number="49" name="Reference" color="13" fill="1" visible="no" active="yes"/>
 <layer number="50" name="dxf" color="7" fill="1" visible="no" active="yes"/>
-<layer number="51" name="tDocu" color="6" fill="1" visible="yes" active="yes"/>
+<layer number="51" name="tDocu" color="6" fill="1" visible="no" active="yes"/>
 <layer number="52" name="bDocu" color="7" fill="1" visible="no" active="yes"/>
 <layer number="53" name="tGND_GNDA" color="7" fill="9" visible="no" active="no"/>
@@
 <layer number="225" name="225bmp" color="7" fill="1" visible="no" active="yes"/>
 <layer number="226" name="226bmp" color="7" fill="1" visible="no" active="yes"/>
-<layer number="227" name="LAYER_2" color="11" fill="1" visible="yes" active="yes"/>
-<layer number="228" name="LAYER_3" color="10" fill="1" visible="yes" active="yes"/>
-<layer number="229" name="LAYER_4" color="14" fill="1" visible="yes" active="yes"/>
-<layer number="230" name="LAYER_5" color="12" fill="1" visible="yes" active="yes"/>
-<layer number="231" name="LAYER_6" color="9" fill="1" visible="yes" active="yes"/>
+<layer number="227" name="LAYER_2" color="11" fill="1" visible="no" active="yes"/>
+<layer number="228" name="LAYER_3" color="10" fill="1" visible="no" active="yes"/>
+<layer number="229" name="LAYER_4" color="14" fill="1" visible="no" active="yes"/>
+<layer number="230" name="LAYER_5" color="12" fill="1" visible="no" active="yes"/>
+<layer number="231" name="LAYER_6" color="9" fill="1" visible="no" active="yes"/>
+<layer number="232" name="Eagle3D_PG2" color="7" fill="1" visible="no" active="yes"/>
+<layer number="233" name="Eagle3D_PG3" color="7" fill="1" visible="no" active="yes"/>
 <layer number="248" name="Housing" color="7" fill="1" visible="no" active="yes"/>
 <layer number="249" name="Edge" color="7" fill="1" visible="no" active="yes"/>
@@
 <attribute name="VALUE" x="14.704" y="24.2" size="1.016" layer="27" rot="R180"/>
 </element>
-<element name="JP1" library="Testing" package="1X01_OFFSET_SMALL" value="" x="2.54" y="1.27" smashed="yes" rot="R90">
+<element name="JP1" library="Testing" package="1X08_OFFSET_REDUCED" value="" x="2.54" y="1.27" smashed="yes" rot="R90">
 <attribute name="VALUE" x="6.35" y="0" size="1.27" layer="27" rot="R90"/>
 </element>
-<element name="JP2" library="Testing" package="1X01_OFFSET_SMALL" value="" x="17.78" y="19.05" smashed="yes" rot="R270">
+<element name="JP2" library="Testing" package="1X08_OFFSET_REDUCED" value="" x="17.78" y="19.05" smashed="yes" rot="R270">
 <attribute name="VALUE" x="13.97" y="20.32" size="1.27" layer="27" rot="R270"/>
 </element>
@@
 <contactref element="C3" pad="C"/>
 <contactref element="C2" pad="2"/>
-<contactref element="JP1" pad="P$1"/>
-<contactref element="JP2" pad="P$8"/>
-<contactref element="JP1" pad="P$6"/>
+<contactref element="JP1" pad="1"/>
+<contactref element="JP2" pad="8"/>
+<contactref element="JP1" pad="6"/>
 <wire x1="6.504" y1="6.615" x2="6.504" y2="7.265" width="0.254" layer="1"/>
 <wire x1="6.504" y1="10.515" x2="6.504" y2="11.165" width="0.254" layer="1"/>
@@
 <contactref element="U1" pad="2"/>
 <contactref element="U1" pad="1"/>
-<contactref element="JP1" pad="P$5"/>
+<contactref element="JP1" pad="5"/>
 <wire x1="6.35" y1="12.1412" x2="6.7564" y2="12.1412" width="0.9144" layer="1"/>
 <wire x1="6.7564" y1="12.1412" x2="6.7818" y2="12.1158" width="0.9144" layer="1"/>
@@
 <contactref element="U1" pad="6"/>
 <contactref element="U1" pad="5"/>
-<contactref element="JP1" pad="P$4"/>
+<contactref element="JP1" pad="4"/>
 <wire x1="6.35" y1="9.5504" x2="6.7564" y2="9.5504" width="0.9144" layer="1"/>
 <wire x1="6.7564" y1="9.5504" x2="6.7818" y2="9.525" width="0.9144" layer="1"/>
@@
 <contactref element="U1" pad="8"/>
 <contactref element="U1" pad="7"/>
-<contactref element="JP1" pad="P$3"/>
+<contactref element="JP1" pad="3"/>
 <wire x1="6.35" y1="8.2296" x2="6.7818" y2="8.2296" width="0.9144" layer="1"/>
 <wire x1="6.504" y1="8.0756" x2="6.504" y2="7.915" width="0.254" layer="1"/>
@@
 <contactref element="U1" pad="12"/>
 <contactref element="U1" pad="11"/>
-<contactref element="JP1" pad="P$2"/>
+<contactref element="JP1" pad="2"/>
 <wire x1="6.35" y1="5.6388" x2="6.7818" y2="5.6388" width="0.9144" layer="1"/>
 <wire x1="6.504" y1="5.4848" x2="6.504" y2="5.315" width="0.254" layer="1"/>
@@
 <contactref element="C1" pad="1"/>
 <contactref element="C3" pad="A"/>
-<contactref element="JP1" pad="P$8"/>
+<contactref element="JP1" pad="8"/>
 <wire x1="8.89" y1="16.51" x2="8.51" y2="16.51" width="0.9144" layer="1"/>
 <wire x1="10.668" y1="14.732" x2="8.89" y2="16.51" width="0.9144" layer="1"/>
@@
 <signal name="VCC">
 <contactref element="U1" pad="20"/>
-<contactref element="JP1" pad="P$7"/>
+<contactref element="JP1" pad="7"/>
 <contactref element="C2" pad="1"/>
 <wire x1="9.54" y1="13.97" x2="9.54" y2="14.59" width="0.254" layer="1"/>
@@
 <signal name="PWMA">
 <contactref element="U1" pad="23"/>
-<contactref element="JP2" pad="P$1"/>
+<contactref element="JP2" pad="1"/>
 <wire x1="13.816" y1="11.815" x2="14.609" y2="11.815" width="0.254" layer="1"/>
 <wire x1="14.609" y1="11.815" x2="14.9606" y2="12.1666" width="0.254" layer="1"/>
@@
 <signal name="AIN2">
 <contactref element="U1" pad="22"/>
-<contactref element="JP2" pad="P$2"/>
+<contactref element="JP2" pad="2"/>
 <wire x1="13.816" y1="11.165" x2="14.848" y2="11.165" width="0.254" layer="1"/>
 <wire x1="14.848" y1="11.165" x2="15.494" y2="11.811" width="0.254" layer="1"/>
@@
 <signal name="AIN1">
 <contactref element="U1" pad="21"/>
-<contactref element="JP2" pad="P$3"/>
+<contactref element="JP2" pad="3"/>
 <wire x1="13.97" y1="13.97" x2="17.78" y2="13.97" width="0.254" layer="16"/>
 <wire x1="12.2682" y1="12.2682" x2="13.97" y2="13.97" width="0.254" layer="16"/>
@@
 <signal name="STBY">
 <contactref element="U1" pad="19"/>
-<contactref element="JP2" pad="P$4"/>
+<contactref element="JP2" pad="4"/>
 <wire x1="13.816" y1="9.215" x2="14.676" y2="9.215" width="0.254" layer="1"/>
 <wire x1="14.676" y1="9.215" x2="15.24" y2="9.779" width="0.254" layer="1"/>
@@
 <signal name="BIN1">
 <contactref element="U1" pad="17"/>
-<contactref element="JP2" pad="P$5"/>
+<contactref element="JP2" pad="5"/>
 <wire x1="13.816" y1="7.915" x2="14.9" y2="7.915" width="0.254" layer="1"/>
 <wire x1="14.9" y1="7.915" x2="15.875" y2="8.89" width="0.254" layer="1"/>
@@
 <signal name="BIN2">
 <contactref element="U1" pad="16"/>
-<contactref element="JP2" pad="P$6"/>
+<contactref element="JP2" pad="6"/>
 <wire x1="13.816" y1="7.265" x2="15.595" y2="7.265" width="0.254" layer="1"/>
 <wire x1="15.595" y1="7.265" x2="16.51" y2="6.35" width="0.254" layer="1"/>
@@
 <signal name="PWMB">
 <contactref element="U1" pad="15"/>
-<contactref element="JP2" pad="P$7"/>
+<contactref element="JP2" pad="7"/>
 <wire x1="13.816" y1="6.615" x2="14.975" y2="6.615" width="0.254" layer="1"/>
 <wire x1="14.975" y1="6.615" x2="15.24" y2="6.35" width="0.254" layer="1"/>
