File: Hardware/SparkFun_Motor_Driver-TB6612FNG.sch (EAGLE design)
At the start: 10 parts, among them U1 TB6621FNG

Commit message: Update IC Value
Regarding this issue [ https://github.com/sparkfun/Motor_Driver-Dual_TB6612FNG/issues/1 ].

The part used in the board layout and schematic files was incorrectly labeled as TB6621FNG. The value should actually be labeled as TB6612FNG.
Parts:
- U1: value TB6621FNG -> TB6612FNG
Changed lines of the file:
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@@
 <?xml version="1.0" encoding="utf-8"?>
 <!DOCTYPE eagle SYSTEM "eagle.dtd">
-<eagle version="7.5.0">
+<eagle version="7.6.0">
 <drawing>
 <settings>
@@
 <layer number="254" name="cooling" color="7" fill="1" visible="yes" active="yes"/>
 </layers>
-<schematic xreflabel="%F%N/%S" xrefpart="/%S">
+<schematic xreflabel="%F%N/%S" xrefpart="/%S.%C%R">
 <attributes>
 </attributes>
@@
 <parts>
 <part name="FRAME1" library="SparkFun" deviceset="FRAME-LETTER" device=""/>
-<part name="U1" library="SparkFun" deviceset="TB6621FNG" device=""/>
+<part name="U1" library="SparkFun" deviceset="TB6621FNG" device="" value="TB6612FNG"/>
 <part name="C1" library="SparkFun" deviceset="CAP" device="0402-CAP" value="0.1uF"/>
 <part name="C2" library="SparkFun" deviceset="CAP" device="0402-CAP" value="0.1uF"/>
